Commit message: changed the mass of the lidar

File: velodyne_description/urdf/VLP-16.urdf.xacro (robot description, xacro)
@@ -10,5 +10,5 @@
     <link name="${name}_base_link">
       <inertial>
-        <mass value="0.83"/>
+        <mass value="0.1"/>
         <origin xyz="0 0 0.03585"/>
         <inertia ixx="${(0.83 * (3.0*0.0516*0.0516 + 0.0717*0.0717)) / 12.0}" ixy="0" ixz="0"

Commit message: modified timestamp and specs

File: velodyne_description/urdf/VLP-16.urdf.xacro (robot description, xacro)
@@ -10,9 +10,9 @@
     <link name="${name}_base_link">
       <inertial>
-        <mass value="0.1"/>
+        <mass value="0.05"/>
         <origin xyz="0 0 0.03585"/>
-        <inertia ixx="${(0.83 * (3.0*0.0516*0.0516 + 0.0717*0.0717)) / 12.0}" ixy="0" ixz="0"
-          iyy="${(0.83 * (3.0*0.0516*0.0516 + 0.0717*0.0717)) / 12.0}" iyz="0"
-          izz="${0.5 * 0.83 * (0.0516*0.0516)}"/>
+        <inertia ixx="${0.05*(0.83 * (3.0*0.0516*0.0516 + 0.0717*0.0717)) / 12.0}" ixy="0" ixz="0"
+                 iyy="${0.05*(0.83 * (3.0*0.0516*0.0516 + 0.0717*0.0717)) / 12.0}" iyz="0"
+                 izz="${0.05*0.5 * 0.83 * (0.0516*0.0516)}"/>
       </inertial>
       <visual>

Commit message: revert back to original lidar specs

File: velodyne_description/urdf/VLP-16.urdf.xacro (robot description, xacro)
@@ -10,9 +10,9 @@
     <link name="${name}_base_link">
       <inertial>
-        <mass value="0.05"/>
+        <mass value="0.5"/>
         <origin xyz="0 0 0.03585"/>
-        <inertia ixx="${0.05*(0.83 * (3.0*0.0516*0.0516 + 0.0717*0.0717)) / 12.0}" ixy="0" ixz="0"
-                 iyy="${0.05*(0.83 * (3.0*0.0516*0.0516 + 0.0717*0.0717)) / 12.0}" iyz="0"
-                 izz="${0.05*0.5 * 0.83 * (0.0516*0.0516)}"/>
+        <inertia ixx="${(0.83 * (3.0*0.0516*0.0516 + 0.0717*0.0717)) / 12.0}" ixy="0" ixz="0"
+                 iyy="${(0.83 * (3.0*0.0516*0.0516 + 0.0717*0.0717)) / 12.0}" iyz="0"
+                 izz="${0.5 * 0.83 * (0.0516*0.0516)}"/>
       </inertial>
       <visual>
